Commit message: Add depth camera

File: my_robot/urdf/my_robot.xacro (robot description, xacro)
@@ -186,4 +186,11 @@
     </visual>
   </link>
+  <joint type="fixed" name="camera_optical_joint">
+    <origin xyz="0 0 0" rpy="-1.5707 0 -1.5707"/>
+    <parent link="camera"/>
+    <child link="camera_optical"/>
+  </joint>
+  <link name="camera_optical">
+  </link>
   <joint type="fixed" name="hokuyo_joint">
     <origin xyz="0.08 0 0.08" rpy="0 0 0"/>
