Commit message: Add rviz collors to model

File: mapping_bot/urdf/my_robot.xacro (robot description, xacro)
@@ -2,4 +2,5 @@
 <robot name="my_robot" xmlns:xacro="http://www.ros.org/wiki/xacro">
   <xacro:include filename="$(find mapping_bot)/urdf/my_robot.gazebo"/>
+  <xacro:include filename="$(find mapping_bot)/urdf/materials.urdf"/>
   <link name="base_link"></link>
   <joint name="base_link_joint" type="fixed">
@@ -30,4 +31,5 @@
         <box size=".3 .15 .1"/>
       </geometry>
+      <material name="light_grey"/>
     </visual>
   </link>
@@ -61,4 +63,5 @@
         <cylinder radius="0.07" length="0.07"/>
       </geometry>
+      <material name="black"/>
     </visual>
   </link>
@@ -92,4 +95,5 @@
         <cylinder radius="0.07" length="0.07"/>
       </geometry>
+      <material name="black"/>
     </visual>
   </link>
@@ -123,4 +127,5 @@
         <cylinder radius="0.07" length="0.07"/>
       </geometry>
+      <material name="black"/>
     </visual>
   </link>
@@ -154,4 +159,5 @@
         <cylinder radius="0.07" length="0.07"/>
       </geometry>
+      <material name="black"/>
     </visual>
   </link>
@@ -184,4 +190,5 @@
         <box size="0.04 0.04 0.04"/>
       </geometry>
+      <material name="green"/>
     </visual>
   </link>
